File: 3by2-macropad.kicad_sch (KiCad schematic)
At the start: 13 parts, among them U1 Pico

Commit message: Used correct diode
Parts:
- D1, D2, D3, D4, D5, D6: footprint Diode_THT:D_DO-35_SOD27_P7.62mm_Horizontal -> onesemi-1N914:ON_Semiconductor-017AG-08_2016-O-MFG
Changed lines of the file:
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@@
       (effects (font (size 1.27 1.27)) (justify right))
     )
-    (property "Footprint" "Diode_THT:D_DO-35_SOD27_P7.62mm_Horizontal" (at 190.5 73.66 90)
+    (property "Footprint" "onesemi-1N914:ON_Semiconductor-017AG-08_2016-O-MFG" (at 190.5 73.66 90)
       (effects (font (size 1.27 1.27)) hide)
     )
@@
       (effects (font (size 1.27 1.27)) (justify right))
     )
-    (property "Footprint" "Diode_THT:D_DO-35_SOD27_P7.62mm_Horizontal" (at 177.8 73.66 90)
+    (property "Footprint" "onesemi-1N914:ON_Semiconductor-017AG-08_2016-O-MFG" (at 177.8 73.66 90)
       (effects (font (size 1.27 1.27)) hide)
     )
@@
       (effects (font (size 1.27 1.27)) (justify right))
     )
-    (property "Footprint" "Diode_THT:D_DO-35_SOD27_P7.62mm_Horizontal" (at 190.5 48.26 90)
+    (property "Footprint" "onesemi-1N914:ON_Semiconductor-017AG-08_2016-O-MFG" (at 190.5 48.26 90)
       (effects (font (size 1.27 1.27)) hide)
     )
@@
       (effects (font (size 1.27 1.27)) (justify right))
     )
-    (property "Footprint" "Diode_THT:D_DO-35_SOD27_P7.62mm_Horizontal" (at 177.8 48.26 90)
+    (property "Footprint" "onesemi-1N914:ON_Semiconductor-017AG-08_2016-O-MFG" (at 177.8 48.26 90)
       (effects (font (size 1.27 1.27)) hide)
     )
@@
       (effects (font (size 1.27 1.27)) (justify right))
     )
-    (property "Footprint" "Diode_THT:D_DO-35_SOD27_P7.62mm_Horizontal" (at 203.2 48.26 90)
+    (property "Footprint" "onesemi-1N914:ON_Semiconductor-017AG-08_2016-O-MFG" (at 203.2 48.26 90)
       (effects (font (size 1.27 1.27)) hide)
     )
@@
       (effects (font (size 1.27 1.27)) (justify right))
     )
-    (property "Footprint" "Diode_THT:D_DO-35_SOD27_P7.62mm_Horizontal" (at 203.2 73.66 90)
-      (effects (font (size 1.27 1.27)) hide)
-    )
+    (property "Footprint" "onesemi-1N914:ON_Semiconductor-017AG-08_2016-O-MFG" (at 203.2 73.66 90)
+      (effects (font (size 1.27 1.27)) hide)
+    )
